File: board/board.kicad_pcb (KiCad board)
At the start: 2 copper layers, 21 x 13 mm, 1 part

Commit message: initial
Parts:
- added C1: 1uF, Capacitor_SMD:C_0603_1608Metric, F.Cu at (146.7, 99.1)
- added C2: 1uF, Capacitor_SMD:C_0603_1608Metric, F.Cu at (155.8, 97.0)
- added C3: 1uF, Capacitor_SMD:C_0603_1608Metric, F.Cu at (145.8, 94.4)
- added C4: 1uF, Capacitor_SMD:C_0603_1608Metric, F.Cu at (146.7, 102.0)
- added J1: 012_CAN, on_edge:on_edge_2x05_device, F.Cu at (140.0, 96.5)
- added J2: Conn_01x03_Male, Connector_PinHeader_2.54mm:PinHeader_1x03_P2.54mm_Vertical, F.Cu at (159.2, 93.8)
- added R1: 120R, Resistor_SMD:R_0805_2012Metric, F.Cu at (156.2, 94.5)
- added U1: MCP2542FDxMF, Package_SO:SOIC-8_3.9x4.9mm_P1.27mm, F.Cu at (150.3, 94.3)
- moved LOGO1 2.86 mm to (152.7, 100.0)
Routing:
- net GND: track 0.00 -> 44.8 mm, vias 0 -> 22
- net /implementation/VDD: track 0.00 -> 16.3 mm, vias 0 -> 1
- net /implementation/VIO: track 0.00 -> 15.5 mm, vias 0 -> 1
- net /implementation/CANL: track 0.00 -> 6.95 mm
- net /implementation/CANH: track 0.00 -> 6.53 mm
- net /implementation/TX: track 0.00 -> 6.35 mm
- net /implementation/RX: track 0.00 -> 5.60 mm
- added copper zone on B.Cu, net GND
- added copper zone on F.Cu, net GND
Other:
- outline, holes or cut-outs redrawn
- board text added: "osf.012"
- board text added: "osf.b128.v1.0"
