File: board/implementation.kicad_sch (KiCad schematic)
At the start: 0 parts

Commit message: initial
Parts:
- added C1, C2, C3, C4: 1uF, Capacitor_SMD:C_0603_1608Metric, symbol Device:C_Small
- added U1: MCP2542FDT, Package_SO:SOIC-8_3.9x4.9mm_P1.27mm, symbol Interface_CAN_LIN:MCP2542FDxMF
Connections:
- net GND: now also C1.2, C2.2, C3.2, C4.2, U1.2 (VSS), U1.9 (VSS)
- new net CANH: U1.7 (CANH)
- new net CANL: U1.6 (CANL)
- new net RX: U1.4 (RXD)
- new net STBY: U1.8 (STBY)
- new net TX: U1.1 (TXD)
- new net VDD: C3.1, C4.1, U1.3 (VDD)
- new net VIO: C1.1, C2.1, U1.5 (VIO)
Changed lines of the file:
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@@
 (kicad_sch (version 20211123) (generator eeschema)
   (paper "A4")
-  (hierarchical_label "GND" (shape input) (at 194.31 120.65 0)
+  (junction (at 106.68 87.63) (diameter 0) (color 0 0 0 0)
+  )
+  (junction (at 114.3 103.505) (diameter 0) (color 0 0 0 0)
+  )
+  (junction (at 99.06 103.505) (diameter 0) (color 0 0 0 0)
+  )
+  (junction (at 106.68 103.505) (diameter 0) (color 0 0 0 0)
+  )
+  (junction (at 91.44 90.805) (diameter 0) (color 0 0 0 0)
+  )
+  (junction (at 91.44 103.505) (diameter 0) (color 0 0 0 0)
+  )
+  (wire (pts (xy 99.06 90.805) (xy 99.06 95.885))
+    (stroke (width 0) (type default) (color 0 0 0 0))
+  )
+  (wire (pts (xy 137.795 103.505) (xy 137.795 95.885))
+    (stroke (width 0) (type default) (color 0 0 0 0))
+  )
+  (wire (pts (xy 106.68 103.505) (xy 99.06 103.505))
+    (stroke (width 0) (type default) (color 0 0 0 0))
+  )
+  (wire (pts (xy 114.3 95.885) (xy 114.3 87.63))
+    (stroke (width 0) (type default) (color 0 0 0 0))
+  )
+  (wire (pts (xy 114.3 103.505) (xy 106.68 103.505))
+    (stroke (width 0) (type default) (color 0 0 0 0))
+  )
+  (wire (pts (xy 85.09 90.805) (xy 91.44 90.805))
+    (stroke (width 0) (type default) (color 0 0 0 0))
+  )
+  (wire (pts (xy 114.3 100.965) (xy 114.3 103.505))
+    (stroke (width 0) (type default) (color 0 0 0 0))
+  )
+  (wire (pts (xy 123.825 73.025) (xy 135.255 73.025))
+    (stroke (width 0) (type default) (color 0 0 0 0))
+  )
+  (wire (pts (xy 91.44 90.805) (xy 99.06 90.805))
+    (stroke (width 0) (type default) (color 0 0 0 0))
+  )
+  (wire (pts (xy 106.68 87.63) (xy 85.09 87.63))
+    (stroke (width 0) (type default) (color 0 0 0 0))
+  )
+  (wire (pts (xy 150.495 83.185) (xy 163.195 83.185))
+    (stroke (width 0) (type default) (color 0 0 0 0))
+  )
+  (wire (pts (xy 135.255 73.025) (xy 135.255 75.565))
+    (stroke (width 0) (type default) (color 0 0 0 0))
+  )
+  (wire (pts (xy 150.495 88.265) (xy 163.195 88.265))
+    (stroke (width 0) (type default) (color 0 0 0 0))
+  )
+  (wire (pts (xy 91.44 90.805) (xy 91.44 95.885))
+    (stroke (width 0) (type default) (color 0 0 0 0))
+  )
+  (wire (pts (xy 106.68 100.965) (xy 106.68 103.505))
+    (stroke (width 0) (type default) (color 0 0 0 0))
+  )
+  (wire (pts (xy 114.3 87.63) (xy 106.68 87.63))
+    (stroke (width 0) (type default) (color 0 0 0 0))
+  )
+  (wire (pts (xy 81.915 103.505) (xy 91.44 103.505))
+    (stroke (width 0) (type default) (color 0 0 0 0))
+  )
+  (wire (pts (xy 91.44 100.965) (xy 91.44 103.505))
+    (stroke (width 0) (type default) (color 0 0 0 0))
+  )
+  (wire (pts (xy 99.06 100.965) (xy 99.06 103.505))
+    (stroke (width 0) (type default) (color 0 0 0 0))
+  )
+  (wire (pts (xy 99.06 103.505) (xy 91.44 103.505))
+    (stroke (width 0) (type default) (color 0 0 0 0))
+  )
+  (wire (pts (xy 137.795 69.85) (xy 137.795 75.565))
+    (stroke (width 0) (type default) (color 0 0 0 0))
+  )
+  (wire (pts (xy 114.3 103.505) (xy 137.795 103.505))
+    (stroke (width 0) (type default) (color 0 0 0 0))
+  )
+  (wire (pts (xy 123.825 69.85) (xy 137.795 69.85))
+    (stroke (width 0) (type default) (color 0 0 0 0))
+  )
+  (wire (pts (xy 106.68 95.885) (xy 106.68 87.63))
+    (stroke (width 0) (type default) (color 0 0 0 0))
+  )
+  (hierarchical_label "VDD" (shape input) (at 85.09 87.63 180)
+    (effects (font (size 1.27 1.27)) (justify right))
+  )
+  (hierarchical_label "GND" (shape input) (at 81.915 103.505 180)
+    (effects (font (size 1.27 1.27)) (justify right))
+  )
+  (hierarchical_label "CANL" (shape input) (at 163.195 88.265 0)
     (effects (font (size 1.27 1.27)) (justify left))
   )
+  (hierarchical_label "RX" (shape input) (at 125.095 83.185 180)
+    (effects (font (size 1.27 1.27)) (justify right))
+  )
+  (hierarchical_label "VIO" (shape input) (at 85.09 90.805 180)
+    (effects (font (size 1.27 1.27)) (justify right))
+  )
+  (hierarchical_label "VDD" (shape input) (at 123.825 69.85 180)
+    (effects (font (size 1.27 1.27)) (justify right))
+  )
+  (hierarchical_label "STBY" (shape input) (at 125.095 90.805 180)
+    (effects (font (size 1.27 1.27)) (justify right))
+  )
+  (hierarchical_label "VIO" (shape input) (at 123.825 73.025 180)
+    (effects (font (size 1.27 1.27)) (justify right))
+  )
+  (hierarchical_label "CANH" (shape input) (at 163.195 83.185 0)
+    (effects (font (size 1.27 1.27)) (justify left))
+  )
+  (hierarchical_label "TX" (shape input) (at 125.095 80.645 180)
+    (effects (font (size 1.27 1.27)) (justify right))
+  )
+  (symbol (lib_id "Interface_CAN_LIN:MCP2542FDxMF") (at 137.795 85.725 0) (unit 1)
+    (in_bom yes) (on_board yes) (fields_autoplaced)
+    (property "Reference" "U1" (id 0) (at 139.8144 96.52 0)
+      (effects (font (size 1.27 1.27)) (justify left))
+    )
+    (property "Value" "MCP2542FDT" (id 1) (at 139.8144 99.06 0)
+      (effects (font (size 1.27 1.27)) (justify left))
+    )
+    (property "Footprint" "Package_SO:SOIC-8_3.9x4.9mm_P1.27mm" (id 2) (at 137.795 98.425 0)
+      (effects (font (size 1.27 1.27) italic) hide)
+    )
+    (property "Datasheet" "http://ww1.microchip.com/downloads/en/DeviceDoc/MCP2542FD-4FD-MCP2542WFD-4WFD-Data-Sheet20005514B.pdf" (id 3) (at 137.795 85.725 0)
+      (effects (font (size 1.27 1.27)) hide)
+    )
+    (property "MPN" "MCP2542FDT-E/SN" (id 4) (at 137.795 85.725 0)
+      (effects (font (size 1.27 1.27)) hide)
+    )
+    (property "Digi-Key_PN" "MCP2542FDT-E/SNCT-ND" (id 5) (at 137.795 85.725 0)
+      (effects (font (size 1.27 1.27)) hide)
+    )
+    (pin "1")
+    (pin "2")
+    (pin "3")
+    (pin "4")
+    (pin "5")
+    (pin "6")
+    (pin "7")
+    (pin "8")
+    (pin "9")
+  )
+  (symbol (lib_id "Device:C_Small") (at 99.06 98.425 0) (unit 1)
+    (in_bom yes) (on_board yes) (fields_autoplaced)
+    (property "Reference" "C2" (id 0) (at 101.6 97.1612 0)
+      (effects (font (size 1.27 1.27)) (justify left))
+    )
+    (property "Value" "1uF" (id 1) (at 101.6 99.7012 0)
+      (effects (font (size 1.27 1.27)) (justify left))
+    )
+    (property "Footprint" "Capacitor_SMD:C_0603_1608Metric" (id 2) (at 99.06 98.425 0)
+      (effects (font (size 1.27 1.27)) hide)
+    )
+    (property "Datasheet" "~" (id 3) (at 99.06 98.425 0)
+      (effects (font (size 1.27 1.27)) hide)
+    )
+    (pin "1")
+    (pin "2")
+  )
+  (symbol (lib_id "Device:C_Small") (at 106.68 98.425 0) (unit 1)
+    (in_bom yes) (on_board yes) (fields_autoplaced)
+    (property "Reference" "C3" (id 0) (at 109.22 97.1612 0)
+      (effects (font (size 1.27 1.27)) (justify left))
+    )
+    (property "Value" "1uF" (id 1) (at 109.22 99.7012 0)
+      (effects (font (size 1.27 1.27)) (justify left))
+    )
+    (property "Footprint" "Capacitor_SMD:C_0603_1608Metric" (id 2) (at 106.68 98.425 0)
+      (effects (font (size 1.27 1.27)) hide)
+    )
+    (property "Datasheet" "~" (id 3) (at 106.68 98.425 0)
+      (effects (font (size 1.27 1.27)) hide)
+    )
+    (pin "1")
+    (pin "2")
+  )
+  (symbol (lib_id "Device:C_Small") (at 91.44 98.425 0) (unit 1)
+    (in_bom yes) (on_board yes) (fields_autoplaced)
+    (property "Reference" "C1" (id 0) (at 93.98 97.1612 0)
+      (effects (font (size 1.27 1.27)) (justify left))
+    )
+    (property "Value" "1uF" (id 1) (at 93.98 99.7012 0)
+      (effects (font (size 1.27 1.27)) (justify left))
+    )
+    (property "Footprint" "Capacitor_SMD:C_0603_1608Metric" (id 2) (at 91.44 98.425 0)
+      (effects (font (size 1.27 1.27)) hide)
+    )
+    (property "Datasheet" "~" (id 3) (at 91.44 98.425 0)
+      (effects (font (size 1.27 1.27)) hide)
+    )
+    (pin "1")
+    (pin "2")
+  )
+  (symbol (lib_id "Device:C_Small") (at 114.3 98.425 0) (unit 1)
+    (in_bom yes) (on_board yes) (fields_autoplaced)
+    (property "Reference" "C4" (id 0) (at 116.84 97.1612 0)
+      (effects (font (size 1.27 1.27)) (justify left))
+    )
+    (property "Value" "1uF" (id 1) (at 116.84 99.7012 0)
+      (effects (font (size 1.27 1.27)) (justify left))
+    )
+    (property "Footprint" "Capacitor_SMD:C_0603_1608Metric" (id 2) (at 114.3 98.425 0)
+      (effects (font (size 1.27 1.27)) hide)
+    )
+    (property "Datasheet" "~" (id 3) (at 114.3 98.425 0)
+      (effects (font (size 1.27 1.27)) hide)
+    )
+    (pin "1")
+    (pin "2")
+  )
 )
